File: CAD/ESP-DIsplay/esp12e.sch (KiCad schematic (older format))
At the start: 15 parts, among them J301 Conn_01x03_Female, J302 FTDI_Conn, SW301 Reset, SW302 Flash, U301 LD1117S33TR_SOT223, U302 ESP-12E

Commit message: esp12e adc pinsadded, 1117 power module
Connections:
- net +3V3: now also J301.2 (Pin_2); no longer J301.3 (Pin_3)
- net GND: now also J301.3 (Pin_3); no longer J301.2 (Pin_2)
Changed lines of the file:
@@
 L power:GND #PWR0303
 U 1 1 603E1572
-P 2650 4450
-F 0 "#PWR0303" H 2650 4200 50  0001 C CNN
-F 1 "GND" H 2655 4277 50  0000 C CNN
-F 2 "" H 2650 4450 50  0001 C CNN
-F 3 "" H 2650 4450 50  0001 C CNN
-	1    2650 4450
+P 3050 4600
+F 0 "#PWR0303" H 3050 4350 50  0001 C CNN
+F 1 "GND" H 3055 4427 50  0000 C CNN
+F 2 "" H 3050 4600 50  0001 C CNN
+F 3 "" H 3050 4600 50  0001 C CNN
+	1    3050 4600
 	1    0    0    -1
 $EndComp
@@
 	3050 4200 3250 4200
 Wire Wire Line
-	2800 4050 2800 4400
+	3250 4400 3050 4400
 Wire Wire Line
-	2800 4400 3250 4400
+	3050 4400 3050 4600
 Wire Wire Line
-	3250 4300 2650 4300
+	3250 4300 2800 4300
 Wire Wire Line
-	2650 4300 2650 4450
+	2800 4300 2800 4050
 $EndSCHEMATC

Commit message: ESP32 added
Parts:
- removed C301, C303: CP, Capacitor_Tantalum_SMD:CP_EIA-7343-15_Kemet-W, symbol Device:CP
- removed C302, C304, C305: C, Capacitor_SMD:C_1206_3216Metric, symbol Device:C
- removed D301, D302: D_Schottky, Diode_SMD:D_SOD-123, symbol Device:D_Schottky
- removed J301: Conn_01x03_Female, Connector_PinSocket_2.54mm:PinSocket_1x03_P2.54mm_Vertical, symbol Connector:Conn_01x03_Female
- removed J302: FTDI_Conn, Connector_PinSocket_2.54mm:PinSocket_1x06_P2.54mm_Vertical, symbol Connector:Conn_01x06_Female
- removed R301: R, Resistor_SMD:R_0805_2012Metric, symbol Device:R
- removed SW301: Reset, Button_Switch_THT:SW_PUSH_6mm_H5mm, symbol Switch:SW_Push
- removed U301: LD1117S33TR_SOT223, Package_TO_SOT_SMD:SOT-223-3_TabPin2, symbol Regulator_Linear:LD1117S33TR_SOT223
Connections:
- net RESET: now also U302.1 (~RST)
- net CS renamed GPIO0
- no-connect marks 6 -> 4
