File: CAD/Loet-Station/Loet-Station.sch (KiCad schematic (older format))
At the start: 39 parts, among them J101 Weller Tip, J102 Conn_Power, Q101 BC547, Q102 IRF9540N, SW101 SW_On, SW102 SW_Down, SW103 SW_Up, SW104 SW_T3, SW105 SW_T2, SW106 SW_T1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

Commit message: esp32-mini added, pwm driver for 24v
Parts:
- removed R105: R, Resistor_SMD:R_0805_2012Metric, symbol Device:R
- added D?: D_Zener, symbol Device:D_Zener
- added R?: R, symbol Device:R
- R102, R107: value R -> 1k
Other:
- moved on the sheet: R102, R107
Changed lines of the file:
@@
 $Descr A4 11693 8268
 encoding utf-8
-Sheet 1 6
+Sheet 1 7
 Title ""
 Date ""
@@
 L Device:R R102
 U 1 1 603BC651
-P 3300 2100
-F 0 "R102" V 3093 2100 50  0000 C CNN
-F 1 "R" V 3184 2100 50  0000 C CNN
-F 2 "Resistor_SMD:R_0805_2012Metric" V 3230 2100 50  0001 C CNN
-F 3 "~" H 3300 2100 50  0001 C CNN
-	1    3300 2100
+P 3500 2100
+F 0 "R102" V 3293 2100 50  0000 C CNN
+F 1 "1k" V 3384 2100 50  0000 C CNN
+F 2 "Resistor_SMD:R_0805_2012Metric" V 3430 2100 50  0001 C CNN
+F 3 "~" H 3500 2100 50  0001 C CNN
+	1    3500 2100
 	0    1    1    0
-$EndComp
-$Comp
-L Device:R R105
-U 1 1 603BCD99
-P 3600 2350
-F 0 "R105" H 3670 2396 50  0000 L CNN
-F 1 "R" H 3670 2305 50  0000 L CNN
-F 2 "Resistor_SMD:R_0805_2012Metric" V 3530 2350 50  0001 C CNN
-F 3 "~" H 3600 2350 50  0001 C CNN
-	1    3600 2350
-	1    0    0    -1
 $EndComp
 $Comp
 L Device:R R107
 U 1 1 603BD4D6
-P 4300 1500
-F 0 "R107" H 4370 1546 50  0000 L CNN
-F 1 "R" H 4370 1455 50  0000 L CNN
-F 2 "Resistor_SMD:R_0805_2012Metric" V 4230 1500 50  0001 C CNN
-F 3 "~" H 4300 1500 50  0001 C CNN
-	1    4300 1500
-	1    0    0    -1
-$EndComp
-Wire Wire Line
-	3450 2100 3600 2100
-Wire Wire Line
-	3600 2200 3600 2100
-Connection ~ 3600 2100
-Wire Wire Line
-	3600 2100 3750 2100
-Text GLabel 2950 2100 0    50   Input ~ 0
+P 4050 1500
+F 0 "R107" H 4120 1546 50  0000 L CNN
+F 1 "1k" H 4120 1455 50  0000 L CNN
+F 2 "Resistor_SMD:R_0805_2012Metric" V 3980 1500 50  0001 C CNN
+F 3 "~" H 4050 1500 50  0001 C CNN
+	1    4050 1500
+	1    0    0    -1
+$EndComp
+Text GLabel 3150 2100 0    50   Input ~ 0
 PWM
 Wire Wire Line
-	2950 2100 3150 2100
+	3150 2100 3350 2100
 Wire Wire Line
 	4050 1900 4050 1800
@@
 L power:GND #PWR0105
 U 1 1 603E140B
-P 4050 2500
-F 0 "#PWR0105" H 4050 2250 50  0001 C CNN
-F 1 "GND" H 4055 2327 50  0000 C CNN
-F 2 "" H 4050 2500 50  0001 C CNN
-F 3 "" H 4050 2500 50  0001 C CNN
-	1    4050 2500
-	1    0    0    -1
-$EndComp
-Wire Wire Line
-	4050 2300 4050 2500
-$Comp
-L power:GND #PWR0102
-U 1 1 603F934A
-P 3600 2550
-F 0 "#PWR0102" H 3600 2300 50  0001 C CNN
-F 1 "GND" H 3605 2377 50  0000 C CNN
-F 2 "" H 3600 2550 50  0001 C CNN
-F 3 "" H 3600 2550 50  0001 C CNN
-	1    3600 2550
-	1    0    0    -1
-$EndComp
-Wire Wire Line
-	3600 2500 3600 2550
+P 4050 2650
+F 0 "#PWR0105" H 4050 2400 50  0001 C CNN
+F 1 "GND" H 4055 2477 50  0000 C CNN
+F 2 "" H 4050 2650 50  0001 C CNN
+F 3 "" H 4050 2650 50  0001 C CNN
+	1    4050 2650
+	1    0    0    -1
+$EndComp
 Wire Wire Line
 	4050 1800 4300 1800
@@
 	9900 3400 9900 3450
 Connection ~ 9900 3450
+Wire Wire Line
+	4300 1150 4050 1150
+Wire Wire Line
+	4050 1150 4050 1350
+Connection ~ 4300 1150
+Wire Wire Line
+	4050 1800 4050 1650
+Connection ~ 4050 1800
+$Comp
+L Device:D_Zener D?
+U 1 1 603FFB08
+P 4300 1500
+F 0 "D?" V 4254 1580 50  0000 L CNN
+F 1 "D_Zener" V 4345 1580 50  0000 L CNN
+F 2 "" H 4300 1500 50  0001 C CNN
+F 3 "~" H 4300 1500 50  0001 C CNN
+	1    4300 1500
+	0    1    1    0
+$EndComp
+$Comp
+L Device:R R?
+U 1 1 604072AB
+P 4050 2500
+F 0 "R?" H 4120 2546 50  0000 L CNN
+F 1 "R" H 4120 2455 50  0000 L CNN
+F 2 "" V 3980 2500 50  0001 C CNN
+F 3 "~" H 4050 2500 50  0001 C CNN
+	1    4050 2500
+	1    0    0    -1
+$EndComp
+Wire Wire Line
+	4050 2300 4050 2350
+Wire Wire Line
+	3650 2100 3750 2100
 $EndSCHEMATC

Commit message: changed d1 mini pins, optional i2c oled
Parts:
- removed Q101: BC547, Package_TO_SOT_THT:TO-92_Inline, symbol Transistor_BJT:BC547
- removed Q102: IRF9540N, Package_TO_SOT_THT:TO-220-3_Vertical, symbol Transistor_FET:IRF9540N
- removed R101: 10k, Resistor_SMD:R_0805_2012Metric, symbol Device:R
- removed R104: 39k, Resistor_SMD:R_0805_2012Metric, symbol Device:R
- added Q101: BC847, Package_TO_SOT_SMD:SOT-23, symbol Transistor_BJT:BC847
- added Q102: IRF7404, Package_SO:SOIC-8_3.9x4.9mm_P1.27mm, symbol Transistor_FET:IRF7404
- D102: renamed from D?; footprint (none) -> Diode_SMD:D_SOD-123
- R105: renamed from R?; footprint (none) -> Resistor_SMD:R_0805_2012Metric
Connections:
- net labels removed: ADC0
- wire segments 113 -> 108
Changed lines of the file:
@@
 $Descr A4 11693 8268
 encoding utf-8
-Sheet 1 7
+Sheet 1 6
 Title ""
 Date ""
@@
 $EndComp
 $Comp
-L Transistor_FET:IRF9540N Q102
-U 1 1 603A6BEB
-P 4700 1800
-F 0 "Q102" H 4904 1754 50  0000 L CNN
-F 1 "IRF9540N" H 4904 1845 50  0000 L CNN
-F 2 "Package_TO_SOT_THT:TO-220-3_Vertical" H 4900 1725 50  0001 L CIN
-F 3 "http://www.irf.com/product-info/datasheets/data/irf9540n.pdf" H 4700 1800 50  0001 L CNN
-	1    4700 1800
-	1    0    0    1
-$EndComp
-$Comp
-L Transistor_BJT:BC547 Q101
-U 1 1 603A8243
-P 3950 2100
-F 0 "Q101" H 4141 2146 50  0000 L CNN
-F 1 "BC547" H 4141 2055 50  0000 L CNN
-F 2 "Package_TO_SOT_THT:TO-92_Inline" H 4150 2025 50  0001 L CIN
-F 3 "https://www.onsemi.com/pub/Collateral/BC550-D.pdf" H 3950 2100 50  0001 L CNN
-	1    3950 2100
-	1    0    0    -1
-$EndComp
-$Comp
 L Device:R R102
 U 1 1 603BC651
@@
 Wire Wire Line
 	7400 1250 7400 950
-Text GLabel 3750 6050 2    50   Input ~ 0
-TEMP
-$Comp
-L Device:R R101
-U 1 1 60B80E82
-P 3250 6300
-AR Path="/60B80E82" Ref="R101"  Part="1"
-AR Path="/60A4D645/60B19D17/60B80E82" Ref="R?"  Part="1"
-F 0 "R101" H 3320 6346 50  0000 L CNN
-F 1 "10k" H 3320 6255 50  0000 L CNN
-F 2 "Resistor_SMD:R_0805_2012Metric" V 3180 6300 50  0001 C CNN
-F 3 "~" H 3250 6300 50  0001 C CNN
-	1    3250 6300
-	1    0    0    -1
-$EndComp
-$Comp
-L Device:R R104
-U 1 1 60B80E88
-P 3450 6050
-AR Path="/60B80E88" Ref="R104"  Part="1"
-AR Path="/60A4D645/60B19D17/60B80E88" Ref="R?"  Part="1"
-F 0 "R104" V 3243 6050 50  0000 C CNN
-F 1 "39k" V 3334 6050 50  0000 C CNN
-F 2 "Resistor_SMD:R_0805_2012Metric" V 3380 6050 50  0001 C CNN
-F 3 "~" H 3450 6050 50  0001 C CNN
-	1    3450 6050
-	0    1    1    0
-$EndComp
-Wire Wire Line
-	3750 6050 3600 6050
-Wire Wire Line
-	3250 6050 3250 6150
-$Comp
-L power:GND #PWR0101
-U 1 1 60B80E92
-P 3250 6550
-AR Path="/60B80E92" Ref="#PWR0101"  Part="1"
-AR Path="/60A4D645/60B19D17/60B80E92" Ref="#PWR?"  Part="1"
-F 0 "#PWR0101" H 3250 6300 50  0001 C CNN
-F 1 "GND" H 3255 6377 50  0000 C CNN
-F 2 "" H 3250 6550 50  0001 C CNN
-F 3 "" H 3250 6550 50  0001 C CNN
-	1    3250 6550
-	1    0    0    -1
-$EndComp
-Wire Wire Line
-	3250 6450 3250 6550
-Text GLabel 2650 6050 0    50   Input ~ 0
-ADC0
 NoConn ~ 6200 2850
 NoConn ~ 6200 2950
@@
 $EndComp
 Wire Wire Line
-	3300 6050 3250 6050
-Connection ~ 3250 6050
-Wire Wire Line
-	2650 6050 3250 6050
-Wire Wire Line
 	9900 3450 9900 3550
 Wire Wire Line
@@
 Connection ~ 4050 1800
 $Comp
-L Device:D_Zener D?
+L Device:D_Zener D102
 U 1 1 603FFB08
 P 4300 1500
-F 0 "D?" V 4254 1580 50  0000 L CNN
+F 0 "D102" V 4254 1580 50  0000 L CNN
 F 1 "D_Zener" V 4345 1580 50  0000 L CNN
-F 2 "" H 4300 1500 50  0001 C CNN
+F 2 "Diode_SMD:D_SOD-123" H 4300 1500 50  0001 C CNN
 F 3 "~" H 4300 1500 50  0001 C CNN
 	1    4300 1500
@@
 $EndComp
 $Comp
-L Device:R R?
+L Device:R R105
 U 1 1 604072AB
 P 4050 2500
-F 0 "R?" H 4120 2546 50  0000 L CNN
+F 0 "R105" H 4120 2546 50  0000 L CNN
 F 1 "R" H 4120 2455 50  0000 L CNN
-F 2 "" V 3980 2500 50  0001 C CNN
+F 2 "Resistor_SMD:R_0805_2012Metric" V 3980 2500 50  0001 C CNN
 F 3 "~" H 4050 2500 50  0001 C CNN
 	1    4050 2500
@@
 Wire Wire Line
 	3650 2100 3750 2100
+$Comp
+L Transistor_FET:IRF7404 Q102
+U 1 1 604E313E
+P 4700 1800
+F 0 "Q102" H 4905 1846 50  0000 L CNN
+F 1 "IRF7404" H 4905 1755 50  0000 L CNN
+F 2 "Package_SO:SOIC-8_3.9x4.9mm_P1.27mm" H 4900 1725 50  0001 L CIN
+F 3 "http://www.infineon.com/dgdl/irf7404.pdf?fileId=5546d462533600a4015355fa2b5b1b9e" V 4700 1800 50  0001 L CNN
+	1    4700 1800
+	1    0    0    1
+$EndComp
+$Comp
+L Transistor_BJT:BC847 Q101
+U 1 1 604FE51F
+P 3950 2100
+F 0 "Q101" H 4141 2146 50  0000 L CNN
+F 1 "BC847" H 4141 2055 50  0000 L CNN
+F 2 "Package_TO_SOT_SMD:SOT-23" H 4150 2025 50  0001 L CIN
+F 3 "http://www.infineon.com/dgdl/Infineon-BC847SERIES_BC848SERIES_BC849SERIES_BC850SERIES-DS-v01_01-en.pdf?fileId=db3a304314dca389011541d4630a1657" H 3950 2100 50  0001 L CNN
+	1    3950 2100
+	1    0    0    -1
+$EndComp
 $EndSCHEMATC

Commit message: pcb layout loetstation
Parts:
- added J103: Barrel_Jack_Switch, Connector_BarrelJack:BarrelJack_Horizontal, symbol Connector:Barrel_Jack_Switch
Connections:
- net GND: now also J103.2, J103.3
- net VS: now also J103.1
- net T1: now reaches R115.2, R116.1, SW106.1
- net T2: now reaches R114.2, R115.1, SW105.1
- net T3: now reaches R113.2, R114.1, SW104.1
- net TDN: now reaches R111.1, R112.1, SW102.1
- net TON: now reaches R111.2, R117.1, SW101.1
- net TUP: now reaches R112.2, R113.1, SW103.1
Changed lines of the file:
@@
 Connection ~ 9900 1300
-Wire Wire Line
-	9900 800  9900 1300
 Wire Wire Line
 	10100 800  9900 800
@@
 	1    0    0    -1
 $EndComp
+Text GLabel 9450 3450 0    50   Input ~ 0
+T1
+Text GLabel 9450 3050 0    50   Input ~ 0
+T2
+Text GLabel 9450 2600 0    50   Input ~ 0
+T3
+Text GLabel 9450 2150 0    50   Input ~ 0
+TUP
+Text GLabel 9450 1750 0    50   Input ~ 0
+TDN
+Text GLabel 9450 1300 0    50   Input ~ 0
+TON
+Wire Wire Line
+	9900 800  9900 1300
+Wire Wire Line
+	9450 1300 9900 1300
+Wire Wire Line
+	9450 1750 9900 1750
+Wire Wire Line
+	9450 2150 9900 2150
+Wire Wire Line
+	9450 2600 9900 2600
+Wire Wire Line
+	9450 3050 9900 3050
+Wire Wire Line
+	9450 3450 9900 3450
+$Comp
+L Connector:Barrel_Jack_Switch J103
+U 1 1 6088E786
+P 6150 2050
+F 0 "J103" H 5920 2092 50  0000 R CNN
+F 1 "Barrel_Jack_Switch" H 5920 2001 50  0000 R CNN
+F 2 "Connector_BarrelJack:BarrelJack_Horizontal" H 6200 2010 50  0001 C CNN
+F 3 "~" H 6200 2010 50  0001 C CNN
+	1    6150 2050
+	-1   0    0    -1
+$EndComp
+$Comp
+L power:GND #PWR0126
+U 1 1 608904F2
+P 5550 2250
+F 0 "#PWR0126" H 5550 2000 50  0001 C CNN
+F 1 "GND" H 5555 2077 50  0000 C CNN
+F 2 "" H 5550 2250 50  0001 C CNN
+F 3 "" H 5550 2250 50  0001 C CNN
+	1    5550 2250
+	1    0    0    -1
+$EndComp
+$Comp
+L power:VS #PWR0127
+U 1 1 60891AF5
+P 5550 1800
+F 0 "#PWR0127" H 5350 1650 50  0001 C CNN
+F 1 "VS" H 5565 1973 50  0000 C CNN
+F 2 "" H 5550 1800 50  0001 C CNN
+F 3 "" H 5550 1800 50  0001 C CNN
+	1    5550 1800
+	1    0    0    -1
+$EndComp
+Wire Wire Line
+	5550 1800 5550 1950
+Wire Wire Line
+	5550 1950 5850 1950
+Wire Wire Line
+	5850 2050 5750 2050
+Wire Wire Line
+	5550 2050 5550 2250
+Wire Wire Line
+	5850 2150 5750 2150
+Wire Wire Line
+	5750 2150 5750 2050
+Connection ~ 5750 2050
+Wire Wire Line
+	5750 2050 5550 2050
 $EndSCHEMATC
