File: CAD/Loet-Station/oled.sch (KiCad schematic (older format))
At the start: 1 part, among them J501 OLED

Commit message: esp32-mini added, pwm driver for 24v
Connections:
- net labels added: +3.3V
- net labels removed: VCC
Changed lines of the file:
@@
 $Descr A4 11693 8268
 encoding utf-8
-Sheet 5 6
+Sheet 6 7
 Title ""
 Date ""
@@
 	1    0    0    -1
 $EndComp
-$Comp
-L power:VCC #PWR?
-U 1 1 60C872C5
-P 5400 3200
-AR Path="/60C872C5" Ref="#PWR?"  Part="1"
-AR Path="/60C58A4D/60C5A6B7/60C872C5" Ref="#PWR0501"  Part="1"
-F 0 "#PWR0501" H 5400 3050 50  0001 C CNN
-F 1 "VCC" H 5415 3373 50  0000 C CNN
-F 2 "" H 5400 3200 50  0001 C CNN
-F 3 "" H 5400 3200 50  0001 C CNN
-	1    5400 3200
-	1    0    0    -1
-$EndComp
 Wire Wire Line
 	5150 3350 5400 3350
@@
 	-1   0    0    -1
 $EndComp
+$Comp
+L power:+3.3V #PWR?
+U 1 1 603E81BB
+P 5400 3200
+F 0 "#PWR?" H 5400 3050 50  0001 C CNN
+F 1 "+3.3V" H 5415 3373 50  0000 C CNN
+F 2 "" H 5400 3200 50  0001 C CNN
+F 3 "" H 5400 3200 50  0001 C CNN
+	1    5400 3200
+	1    0    0    -1
+$EndComp
 $EndSCHEMATC
