File: CAD/Loet-Station/options.sch (KiCad schematic (older format))
At the start: 0 parts

Commit message: Loet-Station v1
Changed lines of the file:
@@
 $Descr A4 11693 8268
 encoding utf-8
-Sheet 4 7
+Sheet 5 6
 Title ""
 Date ""
@@
 F1 "oled.sch" 50
 $EndSheet
-$Sheet
-S 4900 3950 1200 700
-U 60C877AC
-F0 "extern-lcd" 50
-F1 "extern-lcd.sch" 50
-$EndSheet
 $EndSCHEMATC
